File: electronics/rmc-pizz-arco/rmc-pizz-arco.kicad_pcb (KiCad board)
At the start: 4 copper layers, 74.8 x 80.8 mm, 80 parts, among them J1 PZT, J2 PZT, J3 PZT, J4 PZT, J5 PZT, J6 PZT, J7 DIN-8, J8 PIZZ/ARCO, U1 OPA4191, U2 OPA4191, U3 OPA4191, U4 CD4066B, U5 CD4066B

Commit message: DRC is down to 139 from 252 at the start of this session
Routing:
- net BUFOUT5: track 30.2 -> 27.4 mm, vias 2 -> 4
- net BUFOUT4: track 30.2 -> 27.4 mm, vias 2 -> 4
- net BUFOUT2: track 30.2 -> 27.4 mm, vias 2 -> 4
- net BUFOUT1: track 30.2 -> 27.4 mm, vias 2 -> 4
- net BUFOUT6: track 30.2 -> 27.4 mm, vias 2 -> 4
- net BUFOUT3: track 30.2 -> 27.4 mm, vias 2 -> 4
- net APN6: track 21.4 -> 22.4 mm
- net APN5: track 21.4 -> 22.4 mm
- net APN4: track 21.4 -> 22.4 mm
- net APN3: track 21.4 -> 22.4 mm
- net APN2: track 21.4 -> 22.4 mm
- net APN1: track 21.4 -> 22.4 mm
- net BUFFB6: track 16.0 -> 16.9 mm, vias 0 -> 2
- net BUFFB5: track 16.0 -> 16.9 mm, vias 0 -> 2
- net BUFFB4: track 16.0 -> 16.9 mm, vias 0 -> 2
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