File: electronics/rmc-pizz-arco/rmc-pizz-arco.kicad_pcb (KiCad board)
At the start: 4 copper layers, 78.8 x 81.3 mm, 80 parts, among them J1 PZT, J2 PZT, J3 PZT, J4 PZT, J5 PZT, J6 PZT, J7 DIN-8, J8 PIZZ/ARCO, U1 OPA4191, U2 OPA4191, U3 OPA4191, U4 CD4066B, U5 CD4066B

Commit message: Make the silkscreen legible
Not a DRC error, and worse for it: the reference designators are what an
assembler and a reviewer both work from, and half of them were unreadable.

Three faults, all visible only in a render:

- Adjacent blocks' sub-row designators landed on top of each other. KiCad
  puts a reference above its part, which for an odd channel points straight
  at the previous block's sub-row 2.8mm away. Sub-row designators now go
  towards their own row instead, mirrored by the channel's sign like
  everything else in a block.
- Both bottom legends ran off both edges of the board, which a fab silently
  clips -- taking the polarity warning with it, the one piece of silkscreen
  that exists because there is no reverse-protection diode. They are now
  sized to fit and asserted against the board width rather than trusted, and
  the redundant "POWERED FROM POLY-DRIVE II" is gone now that the supply
  string says the same thing.
- The tail headers lie flat, so their designators sat across their own pads.
  Parked off the ends.

The channel labels move to the quad side of their row, since the sub-row
designators now occupy the other side.

Board unchanged electrically: 0 DRC violations, 0 unconnected, 53 nets and
233 pin connections still matched against design.py.

Co-Authored-By: Claude Opus 5 <noreply@anthropic.com>
Other:
- board text added: "+/-4.5V from Poly-Drive II CHECK POLARITY - NO REVERSE PROTECTION"
- board text removed: "POWERED FROM POLY-DRIVE II +/-4.5V from Poly-Drive II CHECK POLARITY BEFORE FIRST POWER-UP"
